Commit message: IK

File: marco_description/models/marco/marco.xacro (robot description, xacro)
@@ -1,4 +1,4 @@
 <?xml version="1.0"?>
-<robot xmlns:xacro="http://www.ros.org/wiki/xacro" name="firefighter">
+<robot xmlns:xacro="http://www.ros.org/wiki/xacro" name="marco">
   <xacro:property name="L1" value="0.13"/>
   <xacro:property name="L2" value="0.24"/>
@@ -8,4 +8,5 @@
   <xacro:property name="L6" value="0.31"/>
   <xacro:property name="rho" value="0.5"/>
+  <xacro:property name="PI" value="3.14159265358979"/>
   <gazebo>
     <plugin name="gazebo_ros_control" filename="libgazebo_ros_control.so">
@@ -16,5 +17,12 @@
     <self_collide>1</self_collide>
   </gazebo>
-  <link name="world">
+  <link name="world"/>
+  <link name="link0">
+    <visual>
+      <geometry>
+        <cylinder length="0.01" radius="1.0"/>
+      </geometry>
+      <origin xyz="0 0 0.005" rpy="0 0 0"/>
+    </visual>
     <inertial>
       <mass value="1.0" />
@@ -22,21 +30,10 @@
     </inertial>
   </link>
-  <link name="link0">
-    <visual>
-      <geometry>
-        <cylinder length="0.01" radius="1.0"/>
-      </geometry>
-      <origin xyz="0 0 0.005" rpy="0 0 0"/>
-    </visual>
-    <inertial>
-      <mass value="1.0" />
-      <inertia ixx="1.0" ixy="0.0" ixz="0.0" iyy="1.0" iyz="0.0" izz="1.0" />
-    </inertial>
-  </link>
   <link name="link1">
     <visual>
       <geometry>
-        <mesh filename="package://marco_description/meshes/link1.stl" scale="0.1 0.1 0.1"/>
-      </geometry>
+        <mesh filename="package://marco_description/models/marco/meshes/link1.stl" scale="0.1 0.1 0.1"/>
+      </geometry>
+      <origin xyz="0 0 0" rpy="0 0 ${PI / 2}"/>
     </visual>
     <collision>
@@ -55,6 +52,7 @@
     <visual>
       <geometry>
-        <mesh filename="package://marco_description/meshes/link2.stl" scale="0.1 0.1 0.1"/>
-      </geometry>
+        <mesh filename="package://marco_description/models/marco/meshes/link2.stl" scale="0.1 0.1 0.1"/>
+      </geometry>
+      <origin xyz="0 0 0" rpy="0 0 ${PI / 2}"/>
     </visual>
     <collision>
@@ -73,6 +71,7 @@
     <visual>
       <geometry>
-        <mesh filename="package://marco_description/meshes/link3.stl" scale="0.1 0.1 0.1"/>
-      </geometry>
+        <mesh filename="package://marco_description/models/marco/meshes/link3.stl" scale="0.1 0.1 0.1"/>
+      </geometry>
+      <origin xyz="0 0 0" rpy="0 0 ${PI / 2}"/>
     </visual>
     <collision>
@@ -91,6 +90,7 @@
     <visual>
       <geometry>
-        <mesh filename="package://marco_description/meshes/link4.stl" scale="0.1 0.1 0.1"/>
-      </geometry>
+        <mesh filename="package://marco_description/models/marco/meshes/link4.stl" scale="0.1 0.1 0.1"/>
+      </geometry>
+      <origin xyz="0 0 0" rpy="0 0 ${PI / 2}"/>
     </visual>
     <collision>
@@ -109,6 +109,7 @@
     <visual>
       <geometry>
-        <mesh filename="package://marco_description/meshes/link5.stl" scale="0.1 0.1 0.1"/>
-      </geometry>
+        <mesh filename="package://marco_description/models/marco/meshes/link5.stl" scale="0.1 0.1 0.1"/>
+      </geometry>
+      <origin xyz="0 0 0" rpy="0 0 ${PI / 2}"/>
     </visual>
     <collision>
@@ -127,6 +128,7 @@
     <visual>
       <geometry>
-        <mesh filename="package://marco_description/meshes/link6.stl" scale="0.1 0.1 0.1"/>
-      </geometry>
+        <mesh filename="package://marco_description/models/marco/meshes/link6.stl" scale="0.1 0.1 0.1"/>
+      </geometry>
+      <origin xyz="0 0 0" rpy="0 0 ${PI / 2}"/>
     </visual>
     <collision>
@@ -142,9 +144,11 @@
     </inertial>
   </link>
+  <link name="gripper_tip"/>
   <link name="gripper_a">
     <visual>
       <geometry>
-        <mesh filename="package://marco_description/meshes/gripper_a.stl" scale="0.1 0.1 0.1"/>
-      </geometry>
+        <mesh filename="package://marco_description/models/marco/meshes/gripper_a.stl" scale="0.1 0.1 0.1"/>
+      </geometry>
+      <origin xyz="0 0 0" rpy="0 0 ${PI / 2}"/>
     </visual>
     <inertial>
@@ -156,6 +160,7 @@
     <visual>
       <geometry>
-        <mesh filename="package://marco_description/meshes/gripper_b.stl" scale="0.1 0.1 0.1"/>
-      </geometry>
+        <mesh filename="package://marco_description/models/marco/meshes/gripper_b.stl" scale="0.1 0.1 0.1"/>
+      </geometry>
+      <origin xyz="0 0 0" rpy="0 0 ${PI / 2}"/>
     </visual>
     <inertial>
@@ -178,5 +183,5 @@
   <joint name="joint2" type="continuous">
     <origin xyz="0 0 ${L1}" rpy="0 0 0"/>
-    <axis xyz="1 0 0" />
+    <axis xyz="0 -1 0" />
     <dynamics damping="0.5"/>
     <parent link="link1"/>
@@ -185,5 +190,5 @@
   <joint name="joint3" type="continuous">
     <origin xyz="0 0 ${L2}" rpy="0 0 0"/>
-    <axis xyz="1 0 0" />
+    <axis xyz="0 -1 0" />
     <dynamics damping="0.5"/>
     <parent link="link2"/>
@@ -199,5 +204,5 @@
   <joint name="joint5" type="continuous">
     <origin xyz="0 0 ${L4}" rpy="0 0 0"/>
-    <axis xyz="1 0 0" />
+    <axis xyz="0 -1 0" />
     <dynamics damping="0.5"/>
     <parent link="link4"/>
@@ -211,11 +216,16 @@
     <child link="link6"/>
   </joint>
+  <joint name="gripper_fixed" type="fixed">
+    <origin xyz="0 0 ${L6}" rpy="0 0 0"/>
+    <parent link="link6"/>
+    <child link="gripper_tip"/>
+  </joint>
   <joint name="joint_gripper_a" type="fixed">
-    <origin xyz="-0.1 0 0.17" rpy="0 0 0"/>
+    <origin xyz="0 -0.1 0.17" rpy="0 0 0"/>
     <parent link="link6"/>
     <child link="gripper_a"/>
   </joint>
   <joint name="joint_gripper_b" type="fixed">
-    <origin xyz="0.1 0 0.17" rpy="0 0 0"/>
+    <origin xyz="0 0.1 0.17" rpy="0 0 0"/>
     <parent link="link6"/>
     <child link="gripper_b"/>
